Commit message: Add real robot hardware control (mybot_control)

File: mybot_control/description/ros2_control/mybot_ros2_control.xacro (robot description, xacro)
@@ -1,36 +1,37 @@
 <?xml version="1.0"?>
-<robot xmlns:xacro="http://www.ros.org/wiki/xacro" name="mybot">
-    <ros2_control name="RobotSystem" type="system">
-        <hardware>
-            <plugin>mybot_control/MybotHWInterface"</plugin>
-            <param name="left_wheel_name">left_engine_left_wheel_joint</param>
-            <param name="right_wheel_name">right_engine_right_wheel_joint</param>
-            <param name="loop_rate">30</param>
-            <param name="device">/dev/ttyUSB0</param>
-            <param name="baud_rate">57600</param>
-            <param name="timeout_ms">1000</param>
-            <param name="enc_counts_per_rev">2060</param>
-            <param name="pid_p">20</param>
-            <param name="pid_d">12</param>
-            <param name="pid_i">0</param>
-            <param name="pid_o">50</param>
-        </hardware>
-        <!-- ros2_control Common Interfaces -->
-        <joint name="right_engine_right_wheel_joint">
-            <command_interface name="velocity">
-              <param name="min">-1</param>
-              <param name="max">1</param>
-            </command_interface>
-            <state_interface name="position" />
-            <state_interface name="velocity" />
-        </joint>
-        <joint name="left_engine_left_wheel_joint">
-            <command_interface name="velocity">
-              <param name="min">-1</param>
-              <param name="max">1</param>
-            </command_interface>
-            <state_interface name="position" />
-            <state_interface name="velocity" />
-        </joint>
+<robot xmlns:xacro="http://www.ros.org/wiki/xacro">
+  <xacro:macro name="mybot_ros2_control" params="name prefix">
+    <ros2_control name="${name}" type="system">
+      <hardware>
+        <plugin>mybot_control/MybotHWInterface</plugin>
+        <param name="left_wheel_name">left_engine_left_wheel_joint</param>
+        <param name="right_wheel_name">right_engine_right_wheel_joint</param>
+        <param name="loop_rate">30</param>
+        <param name="device">/dev/arduino</param>
+        <param name="baud_rate">57600</param>
+        <param name="timeout_ms">1000</param>
+        <param name="enc_counts_per_rev">2060</param>
+        <param name="pid_p">20</param>
+        <param name="pid_d">12</param>
+        <param name="pid_i">0</param>
+        <param name="pid_o">50</param>
+      </hardware>
+      <joint name="${prefix}left_engine_left_wheel_joint">
+          <command_interface name="velocity">
+            <param name="min">-1</param>
+            <param name="max">1</param>
+          </command_interface>
+        <state_interface name="position"/>
+        <state_interface name="velocity"/>
+      </joint>
+      <joint name="${prefix}right_engine_right_wheel_joint">
+          <command_interface name="velocity">
+            <param name="min">-1</param>
+            <param name="max">1</param>
+          </command_interface>
+        <state_interface name="position"/>
+        <state_interface name="velocity"/>
+      </joint>
     </ros2_control>
+  </xacro:macro>
 </robot>

File: mybot_control/description/urdf/mybot.urdf.xacro (robot description, xacro)
@@ -1,254 +1,13 @@
 <?xml version="1.0"?>
-<robot name="mybot" xmlns:xacro="http://www.ros.org/wiki/xacro">
-  <!-- Include ros2_control Plugins -->
+<!-- Basic differential drive mobile base -->
+<robot xmlns:xacro="http://www.ros.org/wiki/xacro" name="mybot">
+  <xacro:arg name="prefix" default="" />
+  <xacro:include filename="$(find mybot_control)/urdf/mybot_description.urdf.xacro" />
+  <!-- Import Rviz colors -->
+  <xacro:include filename="$(find mybot_control)/urdf/common_properties.xacro" />
+  <!-- Import diffbot ros2_control description -->
   <xacro:include filename="$(find mybot_control)/ros2_control/mybot_ros2_control.xacro" />
-    <xacro:include filename="common_properties.xacro" />
-    <xacro:property name="base_length" value="0.3" />
-    <xacro:property name="base_width" value="0.3" />
-    <xacro:property name="base_height" value="0.1" />
-    <xacro:property name="engine_length" value="0.025" />
-    <xacro:property name="engine_width" value="0.05" />
-    <xacro:property name="engine_height" value="0.025" />
-    <xacro:property name="caster_base_length" value="0.025" />
-    <xacro:property name="caster_base_width" value="0.025" />
-    <xacro:property name="caster_base_height" value="0.025" />
-    <xacro:property name="lidar_base_length" value="0.1" />
-    <xacro:property name="lidar_base_width" value="0.07" />
-    <xacro:property name="lidar_base_height" value="0.03" />
-    <xacro:property name="lidar_radius" value="0.035" />
-    <xacro:property name="lidar_length" value="0.025" />
-    <xacro:property name="wheel_radius" value="0.033" />
-    <xacro:property name="wheel_length" value="0.027" />
-    <link name="base_footprint" />
-    <link name="base_link">
-        <visual>
-            <geometry>
-                <box size="${base_length} ${base_width} ${base_height}" />
-            </geometry>
-            <origin xyz="0 0 ${base_height / 2.0}" rpy="0 0 0" />
-            <material name="blue" />
-        </visual>
-        <collision>
-            <geometry>
-                <box size="${base_length} ${base_width} ${base_height}" />
-            </geometry>
-            <origin xyz="0 0 ${base_height / 2.0}" rpy="0 0 0" />
-        </collision>
-        <xacro:box_inertia m="5.0" l="${2*base_length}" w="${2*base_width}" h="${2*base_height}"
-                           xyz="0 0 ${base_height / 2.0}" rpy="0 0 0" />
-    </link>
-    <link name="caster_base_front_link">
-        <visual>
-            <geometry>
-                <box size="${caster_base_length} ${caster_base_width} ${caster_base_height}" />
-            </geometry>
-            <origin xyz="0 0 0" rpy="0 0 0" />
-            <material name="blue" />
-        </visual>
-        <collision>
-            <geometry>
-                <box size="${caster_base_length} ${caster_base_width} ${caster_base_height}" />
-            </geometry>
-            <origin xyz="0 0 0" rpy="0 0 0" />
-        </collision>
-        <xacro:box_inertia m="5.0" l="${2*caster_base_length}" w="${2*caster_base_width}" h="${2*caster_base_height}"
-                           xyz="0 0 ${caster_base_height / 2.0}" rpy="0 0 0" />
-    </link>
-    <link name="caster_base_back_link">
-        <visual>
-            <geometry>
-                <box size="${caster_base_length} ${caster_base_width} ${caster_base_height}" />
-            </geometry>
-            <origin xyz="0 0 0" rpy="0 0 0" />
-            <material name="blue" />
-        </visual>
-        <collision>
-            <geometry>
-                <box size="${caster_base_length} ${caster_base_width} ${caster_base_height}" />
-            </geometry>
-            <origin xyz="0 0 0" rpy="0 0 0" />
-        </collision>
-        <xacro:box_inertia m="5.0" l="${2*caster_base_length}" w="${2*caster_base_width}" h="${2*caster_base_height}"
-                           xyz="0 0 ${caster_base_height / 2.0}" rpy="0 0 0" />
-    </link>
-    <link name="left_engine_link">
-        <visual>
-            <geometry>
-                <box size="${engine_length} ${engine_width} ${engine_height}" />
-            </geometry>
-            <origin xyz="0 0 0" rpy="0 0 0" />
-            <material name="blue" />
-        </visual>
-        <collision>
-            <geometry>
-                <box size="${engine_length} ${engine_width} ${engine_height}" />
-            </geometry>
-            <origin xyz="0 0 0" rpy="0 0 0" />
-        </collision>
-        <xacro:box_inertia m="5.0" l="${2*engine_length}" w="${2*engine_width}" h="${2*engine_height}"
-                           xyz="0 0 ${engine_height / 2.0}" rpy="0 0 0" />
-    </link>
-    <link name="right_engine_link">
-        <visual>
-            <geometry>
-                <box size="${engine_length} ${engine_width} ${engine_height}" />
-            </geometry>
-            <origin xyz="0 0 0" rpy="0 0 0" />
-            <material name="blue" />
-        </visual>
-        <collision>
-            <geometry>
-                <box size="${engine_length} ${engine_width} ${engine_height}" />
-            </geometry>
-            <origin xyz="0 0 0" rpy="0 0 0" />
-        </collision>
-        <xacro:box_inertia m="5.0" l="${2*engine_length}" w="${2*engine_width}" h="${2*engine_height}"
-                           xyz="0 0 ${engine_height / 2.0}" rpy="0 0 0" />
-    </link>
-    <xacro:macro name="wheel_link" params="prefix">
-        <link name="${prefix}_wheel_link">
-            <visual>
-                <geometry>
-                    <cylinder radius="${wheel_radius}" length="${wheel_length}" />
-                </geometry>
-                <origin xyz="0 0 0" rpy="${pi / 2.0} 0 0" />
-                <material name="grey" />
-            </visual>
-            <collision>
-                <geometry>
-                    <cylinder radius="${wheel_radius}" length="${wheel_length}" />
-                </geometry>
-                <origin xyz="0 0 0" rpy="${pi / 2.0} 0 0" />
-            </collision>
-            <xacro:cylinder_inertia m="1.0" r="${2*wheel_radius}" h="${2*wheel_length}"
-                                    xyz="0 0 0" rpy="${pi / 2.0} 0 0" />
-        </link>
-    </xacro:macro>
-    <xacro:wheel_link prefix="right" />
-    <xacro:wheel_link prefix="left" />
-    <link name="caster_wheel_front_link">
-        <visual>
-            <geometry>
-                <sphere radius="${wheel_radius / 2.0}" />
-            </geometry>
-            <origin xyz="0 0 0" rpy="0 0 0" />
-            <material name="grey" />
-        </visual>
-        <collision>
-            <geometry>
-                <sphere radius="${wheel_radius / 2.0}" />
-            </geometry>
-            <origin xyz="0 0 0" rpy="0 0 0" />
-        </collision>
-        <xacro:sphere_inertia m="0.5" r="${2*wheel_radius / 2.0}"
-                              xyz="0 0 0" rpy="0 0 0" />
-    </link>
-    <link name="caster_wheel_back_link">
-        <visual>
-            <geometry>
-                <sphere radius="${wheel_radius / 2.0}" />
-            </geometry>
-            <origin xyz="0 0 0" rpy="0 0 0" />
-            <material name="grey" />
-        </visual>
-        <collision>
-            <geometry>
-                <sphere radius="${wheel_radius / 2.0}" />
-            </geometry>
-            <origin xyz="0 0 0" rpy="0 0 0" />
-        </collision>
-        <xacro:sphere_inertia m="0.5" r="${2*wheel_radius / 2.0}"
-                              xyz="0 0 0" rpy="0 0 0" />
-    </link>
-    <link name="lidar_base_link">
-        <visual>
-            <geometry>
-                <box size="${lidar_base_length} ${lidar_base_width} ${lidar_base_height}" />
-            </geometry>
-            <origin xyz="0 0 0" rpy="0 0 0" />
-            <material name="grey" />
-        </visual>
-        <collision>
-            <geometry>
-                <box size="${lidar_base_length} ${lidar_base_width} ${lidar_base_height}" />
-            </geometry>
-            <origin xyz="0 0 0" rpy="0 0 0" />
-        </collision>
-        <xacro:box_inertia m="5.0" l="${2*lidar_base_length}" w="${2*lidar_base_width}" h="${2*lidar_base_height}"
-                           xyz="0 0 ${lidar_base_height / 2.0}" rpy="0 0 0" />
-    </link>
-    <link name="lidar_link">
-        <visual>
-            <geometry>
-                <cylinder radius="${lidar_radius}" length="${lidar_length}" />
-            </geometry>
-            <origin xyz="0 0 ${lidar_length / 2.0}" rpy="0 0 0" />
-            <material name="yellow" />
-        </visual>
-        <collision>
-            <geometry>
-                <cylinder radius="${lidar_radius}" length="${lidar_length}" />
-            </geometry>
-            <origin xyz="0 0 ${lidar_length / 2.0}" rpy="0 0 0" />
-        </collision>
-        <xacro:cylinder_inertia m="0.3" r="${2*lidar_radius}" h="${2*lidar_length}"
-                                xyz="0 0 ${lidar_length / 2.0}" rpy="0 0 0" />
-    </link>
-    <joint name="base_joint" type="fixed">
-        <parent link="base_footprint" />
-        <child link="base_link" />
-        <origin xyz="0 0 ${wheel_radius + (engine_height / 2.0)}" rpy="0 0 0"/>
-    </joint>
-    <joint name="base_right_engine_joint" type="fixed">
-        <parent link="base_link" />
-        <child link="right_engine_link" />
-        <origin xyz="0 ${-(base_width - engine_width) / 2.0} ${-(engine_height) / 2.0}" rpy="0 0 0"/>
-    </joint>
-    <joint name="base_left_engine_joint" type="fixed">
-        <parent link="base_link" />
-        <child link="left_engine_link" />
-        <origin xyz="0 ${(base_width - engine_width) / 2.0} ${-(engine_height) / 2.0}" rpy="0 0 0"/>
-    </joint>
-    <joint name="base_caster_base_front_joint" type="fixed">
-        <parent link="base_link" />
-        <child link="caster_base_front_link" />
-        <origin xyz="${base_length / 2.5} 0 ${-(caster_base_height) / 2.0}" rpy="0 0 0"/>
-    </joint>
-    <joint name="base_caster_base_back_joint" type="fixed">
-        <parent link="base_link" />
-        <child link="caster_base_back_link" />
-        <origin xyz="${-base_length / 2.5} 0 ${-(caster_base_height) / 2.0}" rpy="0 0 0"/>
-    </joint>
-    <joint name="right_engine_right_wheel_joint" type="continuous">
-        <parent link="right_engine_link" />
-        <child link="right_wheel_link" />
-        <origin xyz="0 ${-(wheel_length + (engine_height / 2.0))} 0" rpy="0 0 0" />
-        <axis xyz="0 1 0" />
-    </joint>
-    <joint name="left_engine_left_wheel_joint" type="continuous">
-        <parent link="left_engine_link" />
-        <child link="left_wheel_link" />
-        <origin xyz="0 ${(wheel_length + (engine_height / 2.0))} 0" rpy="0 0 0" />
-        <axis xyz="0 1 0" />
-    </joint>
-    <joint name="caster_base_caster_wheel_front_joint" type="fixed">
-        <parent link="caster_base_front_link" />
-        <child link="caster_wheel_front_link" />
-        <origin xyz="0 0 ${-wheel_radius / 2.0}" rpy="0 0 0" />
-    </joint>
-    <joint name="caster_base_caster_wheel_back_joint" type="fixed">
-        <parent link="caster_base_back_link" />
-        <child link="caster_wheel_back_link" />
-        <origin xyz="0 0 ${-wheel_radius / 2.0}" rpy="0 0 0" />
-    </joint>
-    <joint name="base_lidar_base_joint" type="fixed">
-        <parent link="base_link" />
-        <child link="lidar_base_link" />
-        <origin xyz="0 0 ${base_height}" rpy="0 0 0" />
-    </joint>
-    <joint name="lidar_base__lidar_joint" type="fixed">
-        <parent link="lidar_base_link" />
-        <child link="lidar_link" />
-        <origin xyz="${-lidar_base_length / 6.0} 0 ${lidar_base_height / 2.0}" rpy="0 0 0" />
-    </joint>
+  <xacro:mybot prefix="$(arg prefix)" />
+  <xacro:mybot_ros2_control
+    name="MyBot" prefix="$(arg prefix)" />
 </robot>
