Commit message: Update URDF of Robot

File: mybot_description/urdf/mybot.urdf.xacro (robot description, xacro)
@@ -248,13 +248,23 @@
         <origin xyz="0 0 ${-wheel_radius / 2.0}" rpy="0 0 0" />
     </joint>
-    <joint name="base_lidar_base_joint" type="fixed">
+    <!-- <joint name="base_lidar_base_joint" type="fixed">
         <parent link="base_link" />
         <child link="lidar_base_link" />
         <origin xyz="0 0 ${base_height}" rpy="0 0 0" />
-    </joint>
-    <joint name="lidar_base__lidar_joint" type="fixed">
+    </joint>  -->
+    <joint name="base_lidar_base_joint" type="fixed">
+        <parent link="base_link" />
+        <child link="lidar_base_link" />
+        <origin xyz="${base_length / 2.0 - lidar_base_length / 2.0} 0 ${base_height}" rpy="0 0 0" />
+    </joint>
+    <!-- <joint name="lidar_base__lidar_joint" type="fixed">
         <parent link="lidar_base_link" />
         <child link="lidar_link" />
         <origin xyz="${-lidar_base_length / 6.0} 0 ${lidar_base_height / 2.0}" rpy="0 0 0" />
+    </joint>  -->
+    <joint name="lidar_base_lidar_joint" type="fixed">
+        <parent link="lidar_base_link" />
+        <child link="lidar_link" />
+        <origin xyz="0 0 ${lidar_base_height / 2.0}" rpy="0 0 0" />
     </joint>
 </robot>
